File: jackrabbit.kicad_pcb (KiCad board)
At the start: 2 copper layers, 47.6 x 29.2 mm, 62 parts, among them J1 USB_C, J2 PinHeader_2.54mm_02x10, J3 PinHeader_2.54mm_02x04, J4 PinHeader_2.54mm_02x04, J5 PinHeader_2.54mm_01x04, J6 PinHeader_2.54mm_01x03, SW1 SW_Push, SW2 SW_Push, U1 MIC5319-3.3YD5, U2 74LVX245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

Commit message: Continue layout
Parts:
- J2: footprint Connector_PinHeader_2.54mm:PinHeader_2x10_P2.54mm_Horizontal -> jackrabbit:PinHeader_2x10_P2.54mm_Horizontal_NoSilk
- J5: footprint Connector_PinHeader_2.54mm:PinHeader_1x04_P2.54mm_Vertical -> jackrabbit:PinHeader_1x04_P2.54mm_NoSilk
- J6: footprint Connector_PinHeader_2.54mm:PinHeader_1x03_P2.54mm_Vertical -> jackrabbit:PinHeader_1x03_P2.54mm_NoSilk
- moved R7 51.7 mm to (189.9, 123.9)
- moved R8 51.7 mm to (189.9, 122.2)
- moved D1 25.5 mm to (153.3, 111.2)
- moved R14 25.5 mm to (153.3, 111.2)
- moved SW2 20.4 mm to (146.3, 106.4), turned to 0 degrees
- moved J3 11.3 mm to (174.4, 128.8), turned to -90 degrees
- moved J6 7.62 mm to (125.6, 131.0)
- moved C18 2.90 mm to (132.2, 127.2), turned to 90 degrees
- moved Y1 2.70 mm to (128.6, 127.2), turned to 0 degrees
- moved C17 1.83 mm to (124.3, 127.5), turned to 0 degrees
- moved C6 1.80 mm to (137.3, 123.2)
- moved C15 1.27 mm to (130.2, 110.5)
- moved C13 0.51 mm to (137.0, 112.2)
- moved SW1 0.51 mm to (125.2, 106.4)
- moved R11 0.25 mm to (128.6, 124.4)
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Connections:
- net Net-(R4-Pad1) renamed /D+
- net Net-(R5-Pad1) renamed /D-
Routing:
- net +3V3: track 7.20 -> 27.1 mm, vias 3 -> 5
- net /~{OE_A}: track 0.00 -> 14.2 mm, vias 0 -> 2
- net /D-: track 0.00 -> 8.69 mm
- net /D+: track 0.00 -> 7.73 mm
- net /SWDIO: track 6.30 -> 0.00 mm
- net +5V: track 0.00 -> 6.01 mm
- net /~{DIR_OUT_B}: track 0.00 -> 4.06 mm
- net Net-(R11-Pad2): track 1.00 -> 4.89 mm
- net /VREF_ADC: track 1.13 -> 4.57 mm
- net /~{OE_B}: track 0.00 -> 3.39 mm
- net /SWCLK: track 3.00 -> 0.00 mm
- net /~{DIR_OUT_A}: track 1.17 -> 4.06 mm
- net Net-(C17-Pad2): track 0.00 -> 2.58 mm
- net Net-(C18-Pad2): track 7.86 -> 9.72 mm
- net Net-(J1-PadB5): track 0.00 -> 1.45 mm, vias 0 -> 1
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- added copper zone on B.Cu, net +3V3
- added copper zone on F.Cu, net +3V3
Other:
- board text added: "USER"

Commit message: Continue layout
Parts:
- J3, J4: footprint Connector_PinHeader_2.54mm:PinHeader_2x04_P2.54mm_Horizontal -> jackrabbit:PinHeader_2x04_P2.54mm_NoSilk
- R13: moved to B.Cu
- moved D2 32.0 mm to (161.4, 122.8), turned to 90 degrees
- moved R15 32.0 mm to (161.4, 122.8), turned to 90 degrees
- moved D3 29.3 mm to (164.0, 122.8), turned to 90 degrees
- moved R16 29.3 mm to (164.0, 122.8), turned to 90 degrees
- moved J3 28.4 mm to (145.9, 128.8)
- moved D4 26.8 mm to (166.5, 122.8), turned to 90 degrees
- moved R17 26.8 mm to (166.5, 122.8), turned to 90 degrees
- moved R13 8.52 mm to (134.0, 123.2), turned to -90 degrees
- moved R3 4.27 mm to (137.9, 117.5), turned to 0 degrees
- moved C14 3.34 mm to (141.1, 120.6), turned to -90 degrees
- moved C5 3.30 mm to (138.6, 120.6), turned to -90 degrees
- moved J1 2.62 mm to (148.4, 118.1)
- moved D1 2.54 mm to (150.7, 111.2)
- moved H1 2.54 mm to (151.0, 129.5)
- moved H3 2.54 mm to (151.0, 106.7)
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Connections:
- J3 pad 7: unconnected-(J3-Pad7) -> /ADC0
- U4 pad 28: /~{DIR_OUT_B} -> /~{OE_A}
- U4 pad 29: Net-(R7-Pad1) -> /~{DIR_OUT_B}
- U4 pad 30: Net-(R8-Pad1) -> /~{OE_B}
- U4 pad 31: /~{OE_A} -> Net-(R7-Pad1)
- U4 pad 32: /~{OE_B} -> Net-(R8-Pad1)
Routing:
- net /~{DIR_OUT_A}: track 4.06 -> 39.9 mm
- net /~{OE_A}: track 14.2 -> 48.8 mm
- net /~{OE_B}: track 3.39 -> 35.0 mm
- net /~{DIR_OUT_B}: track 4.06 -> 31.5 mm
- net /~{RESET}: track 0.00 -> 24.1 mm, vias 0 -> 2
- net /SWCLK: track 0.00 -> 17.7 mm, vias 0 -> 1
- net +3V3: track 27.1 -> 44.1 mm, vias 5 -> 10
- net /SWDIO: track 0.00 -> 13.7 mm, vias 0 -> 1
- net +1V1: track 4.74 -> 15.0 mm, vias 2 -> 4
- net /USB_D+: track 0.00 -> 4.35 mm
- net Net-(C17-Pad2): track 2.58 -> 6.60 mm
- net GND: track 1.26 -> 4.86 mm, vias 1 -> 4
- net /USB_D-: track 0.00 -> 3.30 mm
- net /D-: track 8.69 -> 6.77 mm
- net /VREF_ADC: track 4.57 -> 6.44 mm
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- added copper zone on F.Cu, net +1V1
- added copper zone on B.Cu, net GND
- added copper zone on F.Cu, net GND
- removed copper zone on B.Cu, net +3V3
Other:
- board size 47.6 x 29.2 mm -> 45.1 x 29.2 mm
- board text added: "RESET"
- board text removed: "USER"
