File: jackrabbit.kicad_pcb (KiCad board)
At the start: 2 copper layers, 45.1 x 29.2 mm, 63 parts, among them J1 USB_C, J2 PinHeader_2.54mm_02x10, J3 PinHeader_2.54mm_02x04, J4 PinHeader_2.54mm_01x03, SW1 SW_Push, SW2 SW_Push, U1 MIC5319-3.3YD5, U2 74LVX245, U3 W25Q16JVSNIQ, U4 RP2040, U5 74LVX245, Y1 ECS-120-18-33-JGN

Commit message: Finish routing all traces
Parts:
- moved R16 23.3 mm to (156.1, 107.4), turned to 90 degrees
- moved R17 22.0 mm to (156.1, 103.4)
- moved R3 18.0 mm to (152.7, 107.2)
- moved D3 18.0 mm to (155.3, 111.1)
- moved D4 18.0 mm to (152.3, 111.1)
- moved H4 18.0 mm to (131.3, 116.8)
- moved J2 18.0 mm to (125.7, 116.8)
- moved R1 18.0 mm to (158.6, 103.4)
- moved R10 18.0 mm to (141.3, 111.6)
- moved R2 18.0 mm to (158.6, 107.4)
- moved R4 18.0 mm to (156.1, 104.4)
- moved R9 18.0 mm to (144.7, 94.5)
- moved U4 18.0 mm to (146.9, 105.4)
- moved Y1 18.0 mm to (141.8, 114.3)
- moved kibuzzard-62E7AE0F 18.0 mm to (140.8, 115.2)
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Routing:
- net +3V3: track 54.5 -> 69.0 mm
- net +5V: track 12.1 -> 18.0 mm
- net Net-(D3-Pad1): track 5.86 -> 11.4 mm
- net Net-(D4-Pad1): track 2.88 -> 8.29 mm
- net +1V1: track 15.0 -> 18.3 mm, vias 4 -> 5
- net /USB_D+: track 4.35 -> 6.66 mm
- net /USB_D-: track 3.30 -> 5.58 mm
- net /D+: track 7.08 -> 8.11 mm
- net /LEDC: track 4.02 -> 3.00 mm
- net /D-: track 6.77 -> 7.77 mm
- net /VREF_ADC: track 6.44 -> 7.33 mm
- net /~{RESET}: track 56.3 -> 56.9 mm
- added copper zone on F.Cu, net +5V
- added copper zone on F.Cu, net /USB_D+
- added copper zone on B.Cu, net /USB_D-
- added copper zone on F.Cu, net /USB_D-

Commit message: Pass DRC
Parts:
- added REF**: OSHW-Symbol_6.7x6mm_SilkScreen, Symbol:OSHW-Symbol_6.7x6mm_SilkScreen, B.Cu at (154.3, 95.2)
- moved C8 1.27 mm to (142.7, 103.0), turned to 180 degrees
- moved C4 1.17 mm to (152.7, 100.7), turned to 0 degrees
- moved C7 0.15 mm to (142.7, 105.8)
Routing:
- net +3V3: track 69.0 -> 74.7 mm
- net /~{USB_BOOT}: track 63.4 -> 65.4 mm
- net GND: track 4.26 -> 2.91 mm, vias 2 -> 127
- net /SWDIO: track 13.4 -> 14.2 mm
- net /LEDC: track 3.00 -> 3.71 mm
- net Net-(D2-Pad1): track 2.63 -> 2.13 mm
- net Net-(D1-Pad1): track 2.63 -> 2.13 mm
- added copper zone on F.Cu, net VUSB

Commit message: Fix unconnected track end DRC warnings
Routing:
- net +3V3: track 74.7 -> 87.9 mm
- net GND: vias 127 -> 129
